File: polly-power.sch (KiCad schematic (older format))
At the start: 49 parts, among them P1 Power, P2 Analog, P3 Digital, P4 Digital, P5 CONN_01X01, P6 CONN_01X01, P7 CONN_01X01, P8 CONN_01X01

Commit message: Tidy up
Connections:
- net -6.5V: now also P1.1 (Pin_1)
- no-connect marks 5 -> 4
Other:
- note added: "Vouta = (Vrefa*Ga)*(Da/2^^n)\nVoutb = (Vrefb*Gb)*(Db/2^^n)\n=======================\nGa,Gb = Gain selection 1x or 2x (1x)\nn = DAC bit resolution (12)\nDa, Db = Digital value of DAC (0-4095)\n=============================\nVouta = [4 * 1 * 0 / 4096 , 4 * 1 * 4095/4096] = [0, 3.9990234375]\nVoutb = [4 * 1 * 0 / 4096 , 4 * 1 * 4095/4096] = [0, 3.9990234375]"
- note removed: "Vouta = (Vrefa*Ga)*(Da/2^^n)\nVoutb = (Vrefb*Gb)*(Db/2^^n)\n\nGa,Gb = Gain selection 1x or 2x (1x)\nn = DAC bit resolution (12)\nDa, Db = Digital value of DAC (0-4095)\n\nVouta = [4 * 1 * 0 / 4096 , 4 * 1 * 4095/4096] = [0, 3.9990234375]\nVoutb = [4 * 1 * 0 / 4096 , 4 * 1 * 4095/4096] = [0, 3.9990234375]"
- moved on the sheet: R?, U?, U?A, U?B

Commit message: Improve
Parts:
- added R5, R6: 1k, Resistor_THT:R_Axial_DIN0207_L6.3mm_D2.5mm_P2.54mm_Vertical, symbol Device:R
- C1, C2, C3, C5, C6, C7, C8: renamed from C?; footprint (none) -> Capacitor_THT:C_Disc_D4.7mm_W2.5mm_P5.00mm
- C4: renamed from C?; value 4.5uF -> 0.33uF; footprint (none) -> Capacitor_THT:CP_Radial_D6.3mm_P2.50mm
- C9: renamed from C?; footprint (none) -> Capacitor_THT:CP_Radial_D6.3mm_P2.50mm
- J1: renamed from J?; footprint (none) -> Connector_PinHeader_2.54mm:PinHeader_2x04_P2.54mm_Vertical
- R1, R10, R11, R12, R13, R14, R15, R16, R17, R2, R3, R4, R7, R8, R9: renamed from R?; footprint (none) -> Resistor_THT:R_Axial_DIN0207_L6.3mm_D2.5mm_P2.54mm_Vertical
- U1: renamed from U?; footprint (none) -> Package_DIP:DIP-14_W7.62mm_Socket_LongPads
- U2: renamed from U?; footprint (none) -> Package_DIP:DIP-8_W7.62mm_Socket_LongPads
- gave numbers to parts that had none: 7
Connections:
- net 6(**) is gone; now on net GND: P4.2 (Pin_2)
- net A0 is gone; now on net GNDA: P2.1 (Pin_1)
- net A1 is gone; now on net CV: P2.2 (Pin_2)
- net A3 is gone; now on net +5VA: P2.4 (Pin_4)
- net GND: now also R5.2, R6.2
- net VOICE_7_SEL: now also R5.1
- net VOICE_8_SEL: now also R6.1
- net +3V3: no longer names the net of P1.4 (Pin_4)
- net A2 renamed NOISE
- net A4(SDA): no longer names the net of P2.5 (Pin_5)
- net A4(SDA): no longer P3.2 (Pin_2)
- net A5(SCL): no longer names the net of P3.1 (Pin_1)
- net A5(SCL): no longer P2.6 (Pin_6)
- net AUDIO_OUT_SUM renamed AUDIO_BUS
- net AUDIO_BUS: now also P2.6 (Pin_6)
- no-connect marks 4 -> 17
Other:
- note added: "10/9/8 Passthrough \nfrom Arduino to voice \ncards (param select)"
- note added: "A4(SDA)"
- note added: "A5(SCL)"
- note added: "From TI datasheet:\n\n8.2.2.2 Cathode and Load Currents\nIn a typical shunt-regulator configuration (see Figure 7), an external resistor, \nRS, is connected between the supply and the cathode of the LM4040. RS \nmust be set properly, as it sets the total current available to supply the load \n(IL) and bias the LM4040 (IZ). In all cases, IZ must stay within a specified \nrange for proper operation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"
- moved on the sheet: C1, C2, U1G, U2C

Commit message: Continue layout
Parts:
- added C10, C11: 47uF, Capacitor_THT:CP_Radial_D6.3mm_P2.50mm, symbol Device:CP1_Small
- added J2: Conn_02x05_Odd_Even, Connector_IDC:IDC-Header_2x05_P2.54mm_Vertical, symbol Connector_Generic:Conn_02x05_Odd_Even
- added P9: Arduino, Socket_Arduino_Uno:Socket_Strip_Arduino_1x08, symbol Connector_Generic:Conn_01x08
- added Q1, Q2: BC547C, Package_TO_SOT_THT:TO-92_Inline, symbol Transistor_BJT:BC547
- added R18: 22, Resistor_THT:R_Axial_DIN0207_L6.3mm_D2.5mm_P7.62mm_Horizontal, symbol Device:R
- added R19: 10k, Resistor_THT:R_Axial_DIN0207_L6.3mm_D2.5mm_P7.62mm_Horizontal, symbol Device:R
- added R20: 47k, Resistor_THT:R_Axial_DIN0207_L6.3mm_D2.5mm_P7.62mm_Horizontal, symbol Device:R
- added R21: 150k, Resistor_THT:R_Axial_DIN0207_L6.3mm_D2.5mm_P7.62mm_Horizontal, symbol Device:R
- C6: footprint Capacitor_THT:C_Disc_D4.7mm_W2.5mm_P5.00mm -> Capacitor_THT:CP_Radial_D6.3mm_P2.50mm
- R1, R10, R11, R12, R13, R14, R15, R17, R2, R3, R4, R5, R6, R7, R8, R9: footprint Resistor_THT:R_Axial_DIN0207_L6.3mm_D2.5mm_P2.54mm_Vertical -> Resistor_THT:R_Axial_DIN0207_L6.3mm_D2.5mm_P7.62mm_Horizontal
- R16: value 500 -> 909; footprint Resistor_THT:R_Axial_DIN0207_L6.3mm_D2.5mm_P2.54mm_Vertical -> Resistor_THT:R_Axial_DIN0207_L6.3mm_D2.5mm_P7.62mm_Horizontal
- U4, U5: footprint Package_TO_SOT_THT:TO-220-3_Horizontal_TabUp -> Package_TO_SOT_THT:TO-220-3_Vertical
- U7, U8: footprint Package_TO_SOT_THT:TO-92_Inline -> Package_TO_SOT_THT:TO-92_Inline_Wide
Connections:
- net +12VA: now also J2.10 (Pin_10), J2.9 (Pin_9), R18.1
- net +5V: now also P9.1 (Pin_1)
- net -12VA: now also J2.1 (Pin_1), J2.2 (Pin_2); no longer U3.7 (VEE)
- net 2: now also P9.3 (Pin_3)
- net 3(**): now also P9.4 (Pin_4)
- net 4: now also P9.5 (Pin_5)
- net 7: now also P9.7 (Pin_7)
- net GND: now also U3.7 (VEE), P9.2 (Pin_2); no longer P4.2 (Pin_2), U3.6 (~E), U6.9 (~SHDN~)
- net GNDA: now also U6.9 (~SHDN~), C10.2, J2.3 (Pin_3), J2.4 (Pin_4), J2.5 (Pin_5), J2.6 (Pin_6), J2.7 (Pin_7), J2.8 (Pin_8), Q1.3 (E), Q2.2 (B)
- net NOISE: now also Q1.1 (C), R19.2, R21.1
- new net: C11.1, Q2.3 (E), R20.2
- new net: C10.1, R18.2, R19.1, R20.1
- new net: C11.2, Q1.2 (B), R21.2
- new net 6(**): P4.2 (Pin_2), P9.6 (Pin_6), U3.6 (~E)
Other:
- note added: "Noise (YuSynth)\nhttps://yusynth.net/Modular/EN/NOISE/index.html"
- moved on the sheet: C3, C6, C9, R10, R11, R13, R14, R15, R16, R17, R5, R6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
