File: polly-power.kicad_pcb (KiCad board)
At the start: 2 copper layers, 134.7 x 53.3 mm, 53 parts, among them J1 Conn_02x04_Odd_Even, J2 Conn_02x05_Odd_Even, P1 Power, P2 Analog, P3 Digital, P4 Digital, P5 CONN_01X01, P6 CONN_01X01, P7 CONN_01X01, P8 CONN_01X01, P9 Arduino, Q1 BC547C, Q2 BC547C, U1 74LS04, U2 TL072, U3 74HC4051, U4 LM7805_TO220, U5 LM337_TO220, U6 MCP4922-EP, U7 MCP1541-TO, U8 LM4040LP-4.1

Commit message: Split schematic into sheets
Parts:
- added J3: Conn_01x08, Connector_PinHeader_2.54mm:PinHeader_1x08_P2.54mm_Vertical, F.Cu at (235.6, 21.5)
- added J4: Conn_01x08, Connector_PinHeader_2.54mm:PinHeader_1x08_P2.54mm_Vertical, F.Cu at (29.7, 132.6)
- added J5: Conn_02x04_Odd_Even, Connector_PinHeader_2.54mm:PinHeader_2x04_P2.54mm_Vertical, F.Cu at (46.1, 132.6)
- added J6: Conn_01x08, Connector_PinHeader_2.54mm:PinHeader_1x08_P2.54mm_Vertical, F.Cu at (81.3, 55.9)
- added J7: Conn_01x08, Connector_PinHeader_2.54mm:PinHeader_1x08_P2.54mm_Vertical, F.Cu at (25.4, 134.6)
- C1, C2: value 100nF -> 47uF; footprint Capacitor_THT:C_Disc_D4.7mm_W2.5mm_P5.00mm -> Capacitor_THT:CP_Radial_D6.3mm_P2.50mm
- C10, C11: value 47uF -> 100nF; footprint Capacitor_THT:CP_Radial_D6.3mm_P2.50mm -> Capacitor_THT:C_Disc_D4.7mm_W2.5mm_P5.00mm
- C3: value 100nF -> 0.33uF; footprint Capacitor_THT:C_Disc_D4.7mm_W2.5mm_P5.00mm -> Capacitor_THT:CP_Radial_D6.3mm_P2.50mm
- C4: value 0.33uF -> 100nF; footprint Capacitor_THT:CP_Radial_D6.3mm_P2.50mm -> Capacitor_THT:C_Disc_D4.7mm_W2.5mm_P5.00mm
- C5, C7: value 100nF -> 10uF; footprint Capacitor_THT:C_Disc_D4.7mm_W2.5mm_P5.00mm -> Capacitor_THT:CP_Radial_D6.3mm_P2.50mm
- C6, C9: value 10uF -> 100nF; footprint Capacitor_THT:CP_Radial_D6.3mm_P2.50mm -> Capacitor_THT:C_Disc_D4.7mm_W2.5mm_P5.00mm
- J1: value Conn_02x04_Odd_Even -> Conn_02x05_Odd_Even; footprint Connector_PinHeader_2.54mm:PinHeader_2x04_P2.54mm_Vertical -> Connector_IDC:IDC-Header_2x05_P2.54mm_Vertical
- J2: value Conn_02x05_Odd_Even -> Conn_01x08; footprint Connector_IDC:IDC-Header_2x05_P2.54mm_Vertical -> Connector_PinHeader_2.54mm:PinHeader_1x08_P2.54mm_Vertical
- P1: value Power -> Arduino
- P2: value Analog -> Power; footprint Socket_Arduino_Uno:Socket_Strip_Arduino_1x06 -> Socket_Arduino_Uno:Socket_Strip_Arduino_1x08
- P3: value Digital -> Analog; footprint Socket_Arduino_Uno:Socket_Strip_Arduino_1x10 -> Socket_Arduino_Uno:Socket_Strip_Arduino_1x06
- P4: footprint Socket_Arduino_Uno:Socket_Strip_Arduino_1x08 -> Socket_Arduino_Uno:Socket_Strip_Arduino_1x10
- P5: value CONN_01X01 -> Digital; footprint Socket_Arduino_Uno:Arduino_1pin -> Socket_Arduino_Uno:Socket_Strip_Arduino_1x08
- P9: value Arduino -> CONN_01X01; footprint Socket_Arduino_Uno:Socket_Strip_Arduino_1x08 -> Socket_Arduino_Uno:Arduino_1pin
- R1: value 1k -> 47k
- R10: value 119 -> 1k
- R11: value 10k -> 1k
- R13: value 500 -> 1k
- R16: value 909 -> 1k
- R17: value 4k -> 1k
- R18: value 22 -> 10k
- R2: value 1k -> 150k
- R20: value 47k -> 1k
- R21: value 150k -> 10k
- R3: value 1k -> 22
- R4: value 1k -> 10k
- R5: value 1k -> 119
- R6: value 1k -> 500
- R8: value 10k -> 4k
- R9: value 10k -> 909
- U1: value 74LS04 -> LM337_TO220; footprint Package_DIP:DIP-14_W7.62mm_Socket_LongPads -> Package_TO_SOT_THT:TO-220-3_Vertical
- U2: value TL072 -> LM7805_TO220; footprint Package_DIP:DIP-8_W7.62mm_Socket_LongPads -> Package_TO_SOT_THT:TO-220-3_Vertical
- U3: value 74HC4051 -> MCP1541-TO; footprint Package_DIP:DIP-16_W7.62mm_Socket_LongPads -> Package_TO_SOT_THT:TO-92_Inline_Wide
- U4: value LM7805_TO220 -> LM4040LP-4.1; footprint Package_TO_SOT_THT:TO-220-3_Vertical -> Package_TO_SOT_THT:TO-92_Inline_Wide
- U5: value LM337_TO220 -> 74LS04; footprint Package_TO_SOT_THT:TO-220-3_Vertical -> Package_DIP:DIP-14_W7.62mm_Socket_LongPads
- U6: value MCP4922-EP -> 74HC4051; footprint Package_DIP:DIP-14_W7.62mm_Socket_LongPads -> Package_DIP:DIP-16_W7.62mm_Socket_LongPads
- U7: value MCP1541-TO -> TL072; footprint Package_TO_SOT_THT:TO-92_Inline_Wide -> Package_DIP:DIP-8_W7.62mm_Socket_LongPads
- U8: value LM4040LP-4.1 -> MCP4922-EP; footprint Package_TO_SOT_THT:TO-92_Inline_Wide -> Package_DIP:DIP-14_W7.62mm_Socket_LongPads
- moved U5 200.9 mm to (251.8, 21.3), turned to 0 degrees
- moved R10 190.4 mm to (245.7, 44.8), turned to 0 degrees
- moved R13 185.4 mm to (234.9, 43.6), turned to 0 degrees
- moved P9 177.6 mm to (250.7, 150.9)
- moved Q2 176.4 mm to (243.3, 153.7)
- moved R12 161.9 mm to (263.0, 29.3), turned to 0 degrees
- moved R17 160.3 mm to (273.8, 21.2), turned to 0 degrees
- moved Q1 157.7 mm to (216.6, 158.2)
- moved R16 153.5 mm to (263.0, 21.2), turned to 0 degrees
- moved C8 149.6 mm to (273.8, 25.3), turned to 0 degrees
- moved P7 143.0 mm to (251.2, 145.2)
- moved R15 138.9 mm to (251.3, 40.7)
- moved J1 136.4 mm to (28.7, 27.0), turned to 0 degrees
- moved R4 132.5 mm to (233.4, 148.4), turned to 0 degrees
- moved U2 130.4 mm to (48.3, 40.6), turned to 90 degrees
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Connections:
- C1 pad 1: +12VA -> Net-(C1-Pad1)
- C10 pad 1: Net-(C10-Pad1) -> -12VA
- C11 pad 1: Net-(C11-Pad1) -> +5VA
- C11 pad 2: Net-(C11-Pad2) -> GNDA
- C2 pad 1: -12VA -> Net-(C2-Pad1)
- C2 pad 2: GNDA -> Net-(C2-Pad2)
- C3 pad 1: +5V -> +12VA
- C3 pad 2: GND -> GNDA
- C4 pad 1: +12VA -> +5VA
- C5 pad 1: +5VA -> GNDA
- C5 pad 2: GNDA -> /Power/-6.5V
- C6 pad 1: /-6.5V -> +5VA
- C7 pad 1: +5VA -> /Power/MCP_VREF_PWR
- C8 pad 1: +5VA -> +5V
- C8 pad 2: GNDA -> GND
- C9 pad 1: /MCP_VREF -> +12VA
- J1 pad 1: /VDIV_REF -> -12VA
- J1 pad 2: /DAC_REF -> -12VA
- J1 pad 3: /LM_VREF -> GNDA
- J1 pad 4: /DAC_REF -> GNDA
- J1 pad 5: /MCP_VREF -> GNDA
- J1 pad 6: /DAC_REF -> GNDA
- J1 pad 7: +5VA -> GNDA
- J1 pad 8: /DAC_REF -> GNDA
- J2 pad 1: -12VA -> GND
- J2 pad 2: -12VA -> +5V
- J2 pad 3: GNDA -> +5VA
- J2 pad 5: GNDA -> /Power/-6.5V
- J2 pad 6: GNDA -> +12VA
- J2 pad 8: GNDA -> -12VA
- P1 pad 1: /-6.5V -> +5V
- P1 pad 2: (no net) -> GND
- P1 pad 3: (no net) -> /2
- P1 pad 4: (no net) -> /3(**)
- P1 pad 5: +5V -> /4
- P1 pad 6: GND -> /6(**)
- P1 pad 7: GND -> /7
- P1 pad 8: (no net) -> unconnected-(P1-Pad8)
- P2 pad 1: GNDA -> /-6.5V
- P2 pad 2: /CV -> /IOREF
- P2 pad 3: /NOISE -> /Reset
- P2 pad 4: +5VA -> unconnected-(P2-Pad4)
- P2 pad 5: (no net) -> +5V
- P2 pad 6: /AUDIO_BUS -> GND
- P3 pad 1: (no net) -> GNDA
- P3 pad 2: (no net) -> /CV
- P3 pad 3: (no net) -> /NOISE
- P3 pad 4: GND -> /+5VA
- P3 pad 5: /13(SCK) -> unconnected-(P3-Pad5)
- P3 pad 6: (no net) -> /AUDIO_BUS
- P4 pad 1: /7 -> unconnected-(P4-Pad1)
- P4 pad 2: /6(**) -> unconnected-(P4-Pad2)
- P4 pad 3: /~{VOICE_6_SEL} -> /AREF
- P4 pad 4: /~{VOICE_5_SEL} -> GND
- P4 pad 5: /~{VOICE_4_SEL} -> /13(SCK)
- P4 pad 6: /~{VOICE_3_SEL} -> /12(MISO)
- P4 pad 7: /~{VOICE_2_SEL} -> /11(**/MOSI)
- P4 pad 8: /~{VOICE_1_SEL} -> /10(**/SS)
- P5 pad 1: (no net) -> /7
- P6 pad 1: (no net) -> unconnected-(P6-Pad1)
- P7 pad 1: (no net) -> unconnected-(P7-Pad1)
- P8 pad 1: (no net) -> unconnected-(P8-Pad1)
- P9 pad 1: +5V -> unconnected-(P9-Pad1)
- Q1 pad 1: /NOISE -> unconnected-(Q1-Pad1)
- Q1 pad 2: Net-(C11-Pad2) -> GNDA
- Q1 pad 3: GNDA -> Net-(C2-Pad1)
- Q2 pad 1: (no net) -> /NOISE
- Q2 pad 2: GNDA -> Net-(C2-Pad2)
- Q2 pad 3: Net-(C11-Pad1) -> GNDA
- R1 pad 1: /VOICE_1_SEL -> Net-(C1-Pad1)
- R1 pad 2: GND -> Net-(C2-Pad1)
- R10 pad 1: /-6.5V -> /Digital/VOICE_7_SEL
- R10 pad 2: Net-(R10-Pad2) -> GND
- R11 pad 1: Net-(R11-Pad1) -> /Digital/VOICE_8_SEL
- R11 pad 2: /DAC_OUT_B -> GND
- R12 pad 1: /VOICE_6_SEL -> /Digital/VOICE_1_SEL
- R13 pad 1: Net-(R10-Pad2) -> /Digital/VOICE_2_SEL
- R13 pad 2: GNDA -> GND
- R14 pad 1: /AUDIO_OUT -> /Digital/VOICE_3_SEL
- R14 pad 2: /AUDIO_BUS -> GND
- R15 pad 1: +5VA -> /Digital/VOICE_4_SEL
- R15 pad 2: /VDIV_REF -> GND
- R16 pad 1: +5VA -> /Digital/VOICE_5_SEL
- R16 pad 2: /LM_VREF -> GND
- R17 pad 1: /VDIV_REF -> /Digital/VOICE_6_SEL
- R17 pad 2: GNDA -> GND
- R18 pad 1: +12VA -> Net-(R18-Pad1)
- R18 pad 2: Net-(C10-Pad1) -> /DAC and output/DAC_OUT_A
- R19 pad 1: Net-(C10-Pad1) -> Net-(R19-Pad1)
- R19 pad 2: /NOISE -> /DAC and output/DAC_OUT_B
- R2 pad 1: /VOICE_2_SEL -> /NOISE
- R2 pad 2: GND -> Net-(C2-Pad2)
- R20 pad 1: Net-(C10-Pad1) -> /DAC and output/AUDIO_OUT
- R20 pad 2: Net-(C11-Pad1) -> /DAC and output/AUDIO_BUS
- R21 pad 1: /NOISE -> /DAC and output/CV
- R21 pad 2: Net-(C11-Pad2) -> Net-(R18-Pad1)
- R3 pad 1: /VOICE_3_SEL -> +12VA
- R3 pad 2: GND -> Net-(C1-Pad1)
- R4 pad 1: /VOICE_4_SEL -> Net-(C1-Pad1)
- R4 pad 2: GND -> /NOISE
- R5 pad 1: /VOICE_7_SEL -> /Power/-6.5V
- R5 pad 2: GND -> Net-(R5-Pad2)
- R6 pad 1: /VOICE_8_SEL -> Net-(R5-Pad2)
- R6 pad 2: GND -> GNDA
- R7 pad 1: /VOICE_5_SEL -> +5VA
- R7 pad 2: GND -> /Power/VDIV_REF_PWR
- R8 pad 1: /CV -> /Power/VDIV_REF_PWR
- R8 pad 2: Net-(R8-Pad2) -> GNDA
- R9 pad 1: Net-(R8-Pad2) -> +5VA
- R9 pad 2: /DAC_OUT_A -> /Power/LM_VREF_PWR
- U1 pad 1: /VOICE_1_SEL -> Net-(R5-Pad2)
- U1 pad 2: /~{VOICE_1_SEL} -> -12VA
- U1 pad 3: /VOICE_2_SEL -> /Power/-6.5V
- U2 pad 1: /CV -> +12VA
- U2 pad 2: Net-(R8-Pad2) -> GNDA
- U2 pad 3: Net-(R11-Pad1) -> +5VA
- U3 pad 1: /VOICE_5_SEL -> GNDA
- U3 pad 2: /VOICE_7_SEL -> /Power/MCP_VREF_PWR
- U3 pad 3: +5V -> +5VA
- U4 pad 1: +12VA -> (no net)
- U4 pad 2: GNDA -> /Power/LM_VREF_PWR
- U4 pad 3: +5VA -> GNDA
- U5 pad 1: Net-(R10-Pad2) -> /Digital/VOICE_1_SEL
- U5 pad 2: -12VA -> /Digital/~{VOICE_1_SEL}
- U5 pad 3: /-6.5V -> /Digital/VOICE_2_SEL
- U6 pad 1: +5VA -> /Digital/VOICE_5_SEL
- U6 pad 10: /DAC_OUT_B -> /Digital/3(**)
- U6 pad 11: /DAC_REF -> /Digital/2
- U6 pad 12: GNDA -> /Digital/VOICE_4_SEL
- U6 pad 13: /DAC_REF -> /Digital/VOICE_1_SEL
- U6 pad 14: /DAC_OUT_A -> /Digital/VOICE_2_SEL
- U6 pad 2: (no net) -> /Digital/VOICE_7_SEL
- U6 pad 3: /7 -> +5V
- U6 pad 4: /13(SCK) -> /Digital/VOICE_8_SEL
- U6 pad 5: /11(**/MOSI) -> /Digital/VOICE_6_SEL
- U6 pad 6: (no net) -> /Digital/6(**)
- U6 pad 7: (no net) -> GND
- U6 pad 8: GNDA -> GND
- U6 pad 9: GNDA -> /Digital/4
- U7 pad 1: GNDA -> /DAC and output/CV
- U7 pad 2: /MCP_VREF -> Net-(R18-Pad1)
- U7 pad 3: +5VA -> Net-(R19-Pad1)
- U8 pad 1: (no net) -> +5VA
- U8 pad 2: /LM_VREF -> unconnected-(U8-Pad2)
- U8 pad 3: GNDA -> /DAC and output/7
Routing:
- net +5VA: track 225.5 -> 80.9 mm, vias 2 -> 0
- net GNDA: track 312.9 -> 170.3 mm, vias 2 -> 3
- net /NOISE: track 121.6 -> 0.00 mm, vias 4 -> 0
- net GND: track 96.8 -> 0.00 mm
- net /~{VOICE_4_SEL}: track 89.0 -> 0.00 mm, vias 4 -> 0
- net /~{VOICE_5_SEL}: track 79.8 -> 0.00 mm, vias 4 -> 0
- net /~{VOICE_3_SEL}: track 73.9 -> 0.00 mm
- net /~{VOICE_2_SEL}: track 71.2 -> 0.00 mm
- net /~{VOICE_6_SEL}: track 70.7 -> 0.00 mm, vias 4 -> 0
- net /7: track 68.4 -> 0.00 mm, vias 2 -> 0
- net /~{VOICE_1_SEL}: track 67.8 -> 0.00 mm
- net +5V: track 55.1 -> 0.00 mm
- net -12VA: track 20.0 -> 70.0 mm
- net /AUDIO_BUS: track 45.1 -> 0.00 mm, vias 2 -> 0
- net +12VA: track 149.2 -> 106.3 mm
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Other:
- board outline removed
- board text removed: "1"
